File: EPSV-BUG/ESPV-BUG/ESPV-BUG.sch (KiCad schematic (older format))
At the start: 31 parts, among them J1 Conn_01x16_Male, J2 Conn_01x16_Male, J3 Conn_01x05_Female, U1 CH552E, U2 AT25xxx-MA, U3 ESP32-C3, Y1 40MHz, Y2 32k

Commit message: general work
Parts:
- removed J1, J2: Conn_01x16_Male, footprint:01x16_castlations, symbol Connector:Conn_01x16_Male
- added J1, J2: Conn_01x12_Female, footprint:01x12_castlations, symbol Connector:Conn_01x12_Female
- C1, C10, C11, C12, C13, C14, C15, C16, C17, C2, C5, C6, C8: footprint Capacitor_SMD:C_0603_1608Metric_Pad1.05x0.95mm_HandSolder -> Capacitor_SMD:C_0402_1005Metric
- C7: footprint Capacitor_SMD:C_0805_2012Metric_Pad1.15x1.40mm_HandSolder -> Capacitor_SMD:C_0402_1005Metric
- C9: footprint Capacitor_SMD:C_0805_2012Metric_Pad1.15x1.40mm_HandSolder -> Capacitor_SMD:C_0603_1608Metric_Pad1.05x0.95mm_HandSolder
- RN1: footprint Resistor_SMD:R_Array_Convex_4x0603 -> Resistor_SMD:R_Array_Concave_4x0402
- U3: symbol ESP-V-rescue:ESP32-C3-MCU_Espressif-MeshangerV-rescue -> ESPV-BUG-rescue:ESP32-C3-MCU_Espressif-MeshangerV-rescue-ESP-V-rescue
Connections:
- wire segments 203 -> 194
Other:
- note added: "not sure if to use this\n"
