File: EPSV-BUG/ESPV-BUG/ESPV-BUG.kicad_pcb (KiCad board)
At the start: 2 copper layers, 31 parts, among them J1 Conn_01x16_Male, J2 Conn_01x16_Male, J3 Conn_01x05_Female, U1 CH552E, U2 AT25xxx-MA, U3 ESP32-C3, Y1 40MHz, Y2 32k

Commit message: general work
Parts:
- removed C12, C15: 10pF, Capacitor_SMD:C_0603_1608Metric_Pad1.05x0.95mm_HandSolder
- removed C3, C4: 22uF 0805, Capacitor_SMD:C_0805_2012Metric_Pad1.15x1.40mm_HandSolder
- removed C9: 10uF, Capacitor_SMD:C_0805_2012Metric_Pad1.15x1.40mm_HandSolder
- removed Y2: 32k, Crystal:Crystal_DS10_D1.0mm_L4.3mm_Horizontal
- AE1: footprint footprint:ACAG0801-2450-T -> footprint:ACAG0801-2450Trecudedkeepout
- C1, C10, C11, C13, C14, C16, C17, C2, C5, C6, C8: footprint Capacitor_SMD:C_0603_1608Metric_Pad1.05x0.95mm_HandSolder -> Capacitor_SMD:C_0402_1005Metric
- J1: value Conn_01x16_Male -> Conn_01x12_Female; footprint footprint:01x16_castlations -> footprint:01x12_castlations
- J2: value Conn_01x16_Male -> Conn_01x12_Female; footprint footprint:01x16_castlations -> footprint:01x12_castlations; moved to F.Cu
- L1: footprint Inductor_SMD:L_0201_0603Metric -> Inductor_SMD:L_0402_1005Metric
- R1, R2: footprint Resistor_SMD:R_0603_1608Metric_Pad1.05x0.95mm_HandSolder -> Resistor_SMD:R_0402_1005Metric
- RN1: footprint Resistor_SMD:R_Array_Convex_4x0603 -> Resistor_SMD:R_Array_Convex_4x0402
- moved C13 41.0 mm to (172.3, 75.1)
- moved C7 39.5 mm to (170.6, 73.5), turned to 180 degrees
- moved C1 39.5 mm to (166.8, 75.9), turned to 225 degrees
- moved C11 38.4 mm to (172.3, 76.1)
- moved J1 37.5 mm to (179.1, 78.4), turned to 180 degrees
- moved C17 36.6 mm to (171.5, 86.8), turned to 180 degrees
- moved C2 34.6 mm to (166.6, 83.4), turned to 45 degrees
- moved C16 33.5 mm to (173.5, 86.8)
- moved C5 30.1 mm to (170.0, 86.5), turned to 225 degrees
- moved C10 29.5 mm to (175.9, 86.4), turned to 270 degrees
- moved C8 29.0 mm to (174.9, 84.4), turned to 90 degrees
- moved AE1 29.0 mm to (166.8, 90.5)
- moved C6 27.8 mm to (174.9, 86.4), turned to 270 degrees
- moved RN1 26.4 mm to (174.7, 74.9), turned to 90 degrees
- moved U3 26.2 mm to (171.3, 81.3)
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Connections:
- J1 pad 1: +3V3 -> GND
- J1 pad 11: /GP07 -> +3V3
- J1 pad 12: /GP08 -> +3.3VA
- J1 pad 2: +3.3VA -> GND
- J2 pad 10: /GP17 -> /ESP_TX
- J2 pad 11: /ESPUSB- -> GND
- J2 pad 12: /ESPUSB+ -> GND
- J2 pad 2: +3.3VA -> /ESP_RESET
- J2 pad 3: /ESP_RESET -> /GP07
- J2 pad 4: /GP11 -> /GP08
- J2 pad 5: /GP12 -> /BLSEL
- J2 pad 6: /GP13 -> /GP10
- J2 pad 7: /GP14 -> /ESPUSB-
- J2 pad 8: /GP15 -> /ESPUSB+
- J2 pad 9: /GP16 -> /ESP_RX
- U1 pad 10: Net-(U1-Pad10) -> +3V3
Routing:
- net +3V3: track 0.00 -> 44.6 mm, vias 0 -> 3
- net +3.3VA: track 0.00 -> 32.4 mm, vias 0 -> 3
- net /ESP_TX: track 0.00 -> 26.4 mm, vias 0 -> 2
- net /ESP_RX: track 0.00 -> 23.7 mm, vias 0 -> 2
- net /BLSEL: track 0.00 -> 20.4 mm, vias 0 -> 2
- net /GP08: track 0.00 -> 16.3 mm, vias 0 -> 2
- net /GP07: track 0.00 -> 15.8 mm, vias 0 -> 3
- net /CHVP: track 0.00 -> 15.1 mm, vias 0 -> 2
- net /ESP_ENABLE: track 0.00 -> 14.6 mm, vias 0 -> 2
- net /GP10: track 0.00 -> 14.4 mm, vias 0 -> 2
- net /CHUSB-: track 0.00 -> 13.2 mm, vias 0 -> 2
- net /GP06: track 0.00 -> 10.7 mm
- net /GP05: track 0.00 -> 9.47 mm
- net /ESP_RESET: track 0.00 -> 9.39 mm, vias 0 -> 1
- net /GP11: track 0.00 -> 8.68 mm
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- added copper zone on B.Cu, net GND
- added copper zone on F.Cu, net GND
Other:
- board outline added: 16.1 x 25.1 mm
- net class Default: trace_width 0.25 -> 0.2
- net class IO added: clearance 0.15, trace_width 0.2, via_dia 0.65, via_drill 0.35
- net class power added: clearance 0.4, trace_width 0.2, via_dia 0.8, via_drill 0.4
- rule trace_min: 0.2 -> 0.15

Commit message: routing finished ready for silk
Parts:
- added REF**: fHarwin S1001-46 shield clips, footprint:fHarwin S1001-46 shield clips, F.Cu at (177.9, 80.6)
- added REF**: fHarwin S1001-46 shield clips, footprint:fHarwin S1001-46 shield clips, F.Cu at (164.2, 80.4)
- added REF**: fHarwin S1001-46 shield clips, footprint:fHarwin S1001-46 shield clips, F.Cu at (169.1, 87.9)
- J1, J2: footprint footprint:01x12_castlations -> footprint:01x12_pads_2mm; moved to B.Cu
- J3: footprint footprint:01x05_castlations -> footprint:01x5_pads_2mm; moved to B.Cu
- moved J2 0.85 mm to (163.9, 78.3), turned to 180 degrees
- moved J1 0.81 mm to (178.3, 78.3), turned to 0 degrees
- moved J3 0.80 mm to (171.0, 66.3), turned to 90 degrees
Routing:
- net /GP02: track 6.15 -> 9.74 mm, vias 0 -> 1
- net /GP03: track 5.99 -> 8.58 mm, vias 0 -> 1
- net /GP04: track 7.34 -> 9.53 mm, vias 0 -> 1
- net /ESPUSB-: track 4.93 -> 6.73 mm, vias 0 -> 1
- net /GP00: track 5.61 -> 6.92 mm, vias 0 -> 1
- net /GP01: track 5.24 -> 6.51 mm, vias 0 -> 1
- net /ESP_RX: track 23.7 -> 24.9 mm, vias 2 -> 3
- net /ESP_TX: track 26.4 -> 27.4 mm, vias 2 -> 3
- net /ESPUSB+: track 4.92 -> 5.92 mm, vias 0 -> 1
- net +3.3VA: track 32.4 -> 33.2 mm, vias 3 -> 4
- net +3V3: track 44.6 -> 45.3 mm, vias 3 -> 5
- net /CHVP: track 15.1 -> 15.8 mm, vias 2 -> 3
- net /CHUSB+: track 5.82 -> 6.54 mm, vias 2 -> 3
- net /CHBL: track 6.63 -> 7.35 mm, vias 2 -> 3
- net /ESP_ENABLE: track 14.6 -> 15.0 mm, vias 2 -> 3
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Other:
- board text added: "12.7x14.73"
- board text added: "BMI-s-201-c can 13.66 x 12.1"
